File: LT3579-SEPIC-EAGLE-Project/LT3579_SEPIC_Test_Bench.sch (EAGLE design)
At the start: 20 parts, among them IC1 LT3579EFE#PBF, U2 RQ5E050ATTCL

Commit message: Modified Eagle Project and Schematic
Parts:
- removed C_1, C_IN_1, C_IN_2, C_OUT_1, C_OUT_2, C_OUT_3: CGA4J1X7R1E475K125AE, SamacSys_Parts:CGA4J1X7R1E475K125AE
- removed C_C: CGA4F4C0G2W222J085AE, SamacSys_Parts:CGA4F4C0G2W222J085AE
- removed C_F: CGA2B2C0G1H470J050BA, SamacSys_Parts:CGA2B2C0G1H470J050BA
- removed C_SS: CGA4J2X8R1E224K125AE, SamacSys_Parts:CGA4J2X8R1E224K125AE
- removed D1: MBRS360T3G, SamacSys_Parts:MBRS360T3G
- removed IC1: LT3579EFE#PBF, SamacSys_Parts:LT3579EFE#PBF
- removed L1L2: MSD1278T-XXXXX__, MSD1278T-Series:MSD1278T-XXXXX__
- removed R_C: AC0805JR-0712KL, SamacSys_Parts:AC0805JR-0712KL
- removed R_FAULT: AT0805FRE07100KL, AT0805FRE07100KL:AT0805FRE07100KL
- removed R_FB: AC0805FR-07150KL, AC0805FR-07150KL:AC0805FR-07150KL
- removed R_GATE: AC0805DR-0710KL, AC0805DR-0710KL:AC0805DR-0710KL
- removed R_T: AC0805FR-07124KL, SamacSys_Parts:AC0805FR-07124KL
- removed R_UVLO1: AC0805FR-0730KL, AC0805FR-0730KL:AC0805FR-0730KL
- removed R_UVLO2: RT1206BRD075KL, SamacSys_Parts:RT1206BRD075KL
- removed U2: RQ5E050ATTCL, SamacSys_Parts:RQ5E050ATTCL
- added 12P_OUTPUT_CONNECTOR1: CLP-106-02-F-D, SamacSys_Parts:CLP-106-02-F-D
- added 4P_INPUT_CONNECTOR1: SAMTEC-CLP-102-02-X-DJ, SAMTEC-CLP-102-02-X-D:SAMTEC-CLP-102-02-X-DJ
- added C_1_, C_1_1, C_1_2, C_IN_1_, C_IN_1_1, C_IN_1_2, C_IN_2_, C_IN_2_1, C_IN_2_2, C_OUT_1_, C_OUT_1_1, C_OUT_1_2, C_OUT_2_, C_OUT_2_1, C_OUT_2_2, C_OUT_3_, C_OUT_3_1, C_OUT_3_2: CGA4J1X7R1E475K125AE, SamacSys_Parts:CGA4J1X7R1E475K125AE
- added C_C_, C_C_1, C_C_2, C_DECOUPLE_CH_GND_1: CGA4F4C0G2W222J085AE, SamacSys_Parts:CGA4F4C0G2W222J085AE
- added C_DECOUPLE_CH_GND_2: CGADN3X7R1E476M230LE, SamacSys_Parts:CGADN3X7R1E476M230LE
- added C_F_, C_F_1, C_F_2: CGA2B2C0G1H470J050BA, SamacSys_Parts:CGA2B2C0G1H470J050BA
- added C_SS_, C_SS_1, C_SS_2: CGA4J2X8R1E224K125AE, SamacSys_Parts:CGA4J2X8R1E224K125AE
- added D1_, D1_1, D1_2: MBRS360T3G, SamacSys_Parts:MBRS360T3G
- added L1L2_, L1L2_1, L1L2_2: MSD1278T-XXXXX__, MSD1278T-Series:MSD1278T-XXXXX__
- added LT3579_IC_, LT3579_IC_1, LT3579_IC_2: LT3579EFE#PBF, SamacSys_Parts:LT3579EFE#PBF
- added PMOS_, PMOS_1, PMOS_2: RQ5E050ATTCL, SamacSys_Parts:RQ5E050ATTCL
- added R_C_, R_C_1, R_C_2: AC0805JR-0712KL, SamacSys_Parts:AC0805JR-0712KL
- added R_FAULT_, R_FAULT_1, R_FAULT_2: AT0805FRE07100KL, AT0805FRE07100KL:AT0805FRE07100KL
- added R_FB_: AC0805FR-07150KL, AC0805FR-07150KL:AC0805FR-07150KL
- added R_FB_2: AC0805FR-0745K3L, AC0805FR-0745K3L:AC0805FR-0745K3L
- added R_GATE_, R_GATE_1, R_GATE_2: AC0805DR-0710KL, AC0805DR-0710KL:AC0805DR-0710KL
- added R_RB_1: AC0603FR-0764K9L, AC0603FR-0764K9L:AC0603FR-0764K9L
- added R_SHUNT_GND_, R_SHUNT_GND_1, R_SHUNT_GND_2: GMR100HTCFAR100, GMR100HTCFAR100:GMR100HTCFAR100
- added R_T_, R_T_1, R_T_2: AC0805FR-07124KL, SamacSys_Parts:AC0805FR-07124KL
- added R_UVLO1_, R_UVLO1_1, R_UVLO1_2: AC0805FR-0730KL, AC0805FR-0730KL:AC0805FR-0730KL
- added R_UVLO2_, R_UVLO2_1, R_UVLO2_2: RT1206BRD075KL, SamacSys_Parts:RT1206BRD075KL
- added TP_CF_, TP_CF_1, TP_CF_2, TP_CH_GND_, TP_CH_GND_1, TP_CH_GND_2, TP_CLK_, TP_CLK_1, TP_CLK_2, TP_D1_, TP_D1_1, TP_D1_2, TP_FAULT_, TP_FAULT_1, TP_FAULT_2, TP_FB_, TP_FB_1, TP_FB_2, TP_GATE_, TP_GATE_1, TP_GATE_2, TP_GND1_, TP_GND1_1, TP_GND1_2, TP_GND2_, TP_GND2_1, TP_GND2_2, TP_GND3_, TP_GND3_1, TP_GND3_2, TP_GND4_, TP_GND4_1, TP_GND4_2, TP_GND_, TP_GND_1, TP_GND_2, TP_IN_, TP_IN_1, TP_IN_2, TP_OUT_, TP_OUT_1, TP_OUT_2, TP_RT_, TP_RT_1, TP_RT_2, TP_SHDN_, TP_SHDN_1, TP_SHDN_2, TP_SS_, TP_SS_1, TP_SS_2, TP_SW_, TP_SW_1, TP_SW_2: S1751-46R, S1751-46R:S1751-46R
Connections:
- removed net FAULT: R_FAULT.1
- removed net N$10: C_IN_1.1, C_IN_2.1
- removed net N$11: R_FB.2
- removed net N$14: C_SS.1, IC1.SS
- removed net N$8: IC1.RT, R_T.1
- new net CH_GND: 4P_INPUT_CONNECTOR1.2, 4P_INPUT_CONNECTOR1.4, C_DECOUPLE_CH_GND_1.1, C_DECOUPLE_CH_GND_2.1, R_SHUNT_GND_.1, R_SHUNT_GND_1.1, R_SHUNT_GND_2.1
- new net CLK_: 12P_OUTPUT_CONNECTOR1.6, LT3579_IC_.CLKOUT
- new net CLK_1: 12P_OUTPUT_CONNECTOR1.4, LT3579_IC_1.CLKOUT
- new net CLK_2: 12P_OUTPUT_CONNECTOR1.2, LT3579_IC_2.CLKOUT
- new net FAULT_: 12P_OUTPUT_CONNECTOR1.5, LT3579_IC_.!FAULT, R_FAULT_.1
- new net FAULT_1: 12P_OUTPUT_CONNECTOR1.3, LT3579_IC_1.!FAULT, R_FAULT_1.1
- new net FAULT_2: 12P_OUTPUT_CONNECTOR1.1, LT3579_IC_2.!FAULT, R_FAULT_2.1
- new net FB_: LT3579_IC_.FB, R_FB_.2
- new net FB_1: LT3579_IC_1.FB, R_RB_1.2
- new net FB_2: LT3579_IC_2.FB, R_FB_2.2
- new net GATE_: LT3579_IC_.GATE, PMOS_.G, R_GATE_.2
- new net GATE_1: LT3579_IC_1.GATE, PMOS_1.G, R_GATE_1.2
- new net GATE_2: LT3579_IC_2.GATE, PMOS_2.G, R_GATE_2.2
- new net GND: 12P_OUTPUT_CONNECTOR1.10, 12P_OUTPUT_CONNECTOR1.12, 12P_OUTPUT_CONNECTOR1.8, R_SHUNT_GND_.2, R_SHUNT_GND_1.2, R_SHUNT_GND_2.2
- new net RT_: LT3579_IC_.RT, R_T_.1
- new net RT_1: LT3579_IC_1.RT, R_T_1.1
- new net RT_2: LT3579_IC_2.RT, R_T_2.1
- new net SHDN_: LT3579_IC_.!SHDN, R_UVLO1_.1, R_UVLO2_.2
- new net SHDN_1: LT3579_IC_1.!SHDN, R_UVLO1_1.1, R_UVLO2_1.2
- new net SHDN_2: LT3579_IC_2.!SHDN, R_UVLO1_2.1, R_UVLO2_2.2
- new net SS_: C_SS_.1, LT3579_IC_.SS
- new net SS_1: C_SS_1.1, LT3579_IC_1.SS
- new net SS_2: C_SS_2.1, LT3579_IC_2.SS
- new net SW1-2_: C_1_.1, LT3579_IC_.SW1_1, LT3579_IC_.SW1_2, LT3579_IC_.SW1_3, LT3579_IC_.SW1_4, LT3579_IC_.SW1_5, LT3579_IC_.SW2_1, LT3579_IC_.SW2_2, LT3579_IC_.SW2_3, LT3579_IC_.SW2_4, LT3579_IC_.SW2_5
- new net SW1-2_1: C_1_1.1, LT3579_IC_1.SW1_1, LT3579_IC_1.SW1_2, LT3579_IC_1.SW1_3, LT3579_IC_1.SW1_4, LT3579_IC_1.SW1_5, LT3579_IC_1.SW2_1, LT3579_IC_1.SW2_2, LT3579_IC_1.SW2_3, LT3579_IC_1.SW2_4, LT3579_IC_1.SW2_5
- new net SW1-2_2: C_1_2.1, LT3579_IC_2.SW1_1, LT3579_IC_2.SW1_2, LT3579_IC_2.SW1_3, LT3579_IC_2.SW1_4, LT3579_IC_2.SW1_5, LT3579_IC_2.SW2_1, LT3579_IC_2.SW2_2, LT3579_IC_2.SW2_3, LT3579_IC_2.SW2_4, LT3579_IC_2.SW2_5
- new net VC_: C_F_.1, LT3579_IC_.VC, R_C_.1
- new net VC_1: C_F_1.1, LT3579_IC_1.VC, R_C_1.1
- new net VC_2: C_F_2.1, LT3579_IC_2.VC, R_C_2.1
- new net VIN: 4P_INPUT_CONNECTOR1.1, 4P_INPUT_CONNECTOR1.3, C_DECOUPLE_CH_GND_1.2, C_DECOUPLE_CH_GND_2.2, C_IN_1_.1, C_IN_1_1.1, C_IN_1_2.1, C_IN_2_.1, C_IN_2_1.1, C_IN_2_2.1, LT3579_IC_.VIN, LT3579_IC_1.VIN, LT3579_IC_2.VIN, R_FAULT_.2, R_FAULT_1.2, R_FAULT_2.2, R_UVLO1_.2, R_UVLO1_1.2, R_UVLO1_2.2
- new net VOUT_: 12P_OUTPUT_CONNECTOR1.11, C_OUT_1_.1, C_OUT_2_.1, C_OUT_3_.1, PMOS_.S
- new net VOUT_1: 12P_OUTPUT_CONNECTOR1.9, C_OUT_1_1.1, C_OUT_2_1.1, C_OUT_3_1.1, PMOS_1.S
- new net VOUT_2: 12P_OUTPUT_CONNECTOR1.7, C_OUT_1_2.1, C_OUT_2_2.1, C_OUT_3_2.1, PMOS_2.S
- net 0: now also C_C_.2, C_C_1.2, C_C_2.2, C_F_.2, C_F_1.2, C_F_2.2, C_IN_1_.2, C_IN_1_1.2, C_IN_1_2.2, C_IN_2_.2, C_IN_2_1.2, C_IN_2_2.2, C_OUT_1_.2, C_OUT_1_1.2, C_OUT_1_2.2, C_OUT_2_.2, C_OUT_2_1.2, C_OUT_2_2.2, C_OUT_3_.2, C_OUT_3_1.2, C_OUT_3_2.2, C_SS_.2, C_SS_1.2, C_SS_2.2, LT3579_IC_.EPAD, LT3579_IC_1.EPAD, LT3579_IC_2.EPAD, R_T_.2, R_T_1.2, R_T_2.2, R_UVLO2_.1, R_UVLO2_1.1, R_UVLO2_2.1; no longer C_C.2, C_F.2, C_IN_1.2, C_IN_2.2, C_OUT_1.2, C_OUT_2.2, C_OUT_3.2, C_SS.2, R_T.2, R_UVLO2.1
- net N$1: now also C_1_1.2, D1_1.A; no longer R_UVLO1.1, R_UVLO2.2
- net N$13: now also D1_.K, PMOS_.D, R_FB_.1, R_GATE_.1; no longer D1.K, R_FB.1, R_GATE.1, U2.D
- net N$2: now also C_C_1.1, R_C_1.2; no longer R_FAULT.2
- net N$3: now also D1_1.K, PMOS_1.D, R_GATE_1.1, R_RB_1.1; no longer R_GATE.2
- net N$4: now also C_C_.1, R_C_.2; no longer C_C.1, C_F.1, R_C.2
- net N$5: now also C_1_2.2, D1_2.A; no longer C_1.1
- net N$6: now also C_C_2.1, R_C_2.2; no longer C_OUT_1.1, C_OUT_2.1, C_OUT_3.1, U2.S
- net N$7: now also D1_2.K, PMOS_2.D, R_FB_2.1, R_GATE_2.1; no longer R_C.1
- net N$9: now also C_1_.2, D1_.A; no longer C_1.2, D1.A
Other:
- note added: "Connection between board and enclosure and between battery and converter."
- note added: "Connector for all voltage outputs, GNDs, CLK, and Faults."
- note added: "Decoupling capacitors used to reduce voltage ripple from battery input."
- note added: "Ground Test Points"
- note added: "LT3579 SEPIC Config: 13Vin -> 5Vout"
- note added: "LT3579 SEPIC Config: 13Vin -> 6.5Vout"
- note added: "Shunt resistor to measure difference between GNDS."
- note added: "This will mate with the male connector on the enclosure."
- note added: "split the flow of current by having two GND and Vin pins."

Commit message: Modfied Schematic files eagle
Connections:
- net GND: now also LT3579_IC_.SYNC, LT3579_IC_1.SYNC, LT3579_IC_2.SYNC
Changed lines of the file:
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@@
 <setting verticaltext="up"/>
 </settings>
-<grid distance="0.1" unitdist="inch" unit="inch" style="lines" multiple="1" display="yes" altdistance="0.01" altunitdist="inch" altunit="inch"/>
+<grid distance="0.1" unitdist="inch" unit="inch" style="lines" multiple="1" display="no" altdistance="0.01" altunitdist="inch" altunit="inch"/>
 <layers>
 <layer number="1" name="Top" color="4" fill="1" visible="no" active="no"/>
@@
 <wire x1="22.86" y1="-45.72" x2="27.94" y2="-45.72" width="0.1524" layer="91"/>
 <junction x="22.86" y="-35.56"/>
+<junction x="-22.86" y="-2.54"/>
+<junction x="-22.86" y="-5.08"/>
+<junction x="-22.86" y="-7.62"/>
+<junction x="-22.86" y="-10.16"/>
+<junction x="22.86" y="-10.16"/>
+<junction x="22.86" y="-7.62"/>
+<junction x="22.86" y="-5.08"/>
+<junction x="22.86" y="-2.54"/>
 </segment>
 <segment>
@@
 <wire x1="-83.82" y1="-25.4" x2="-83.82" y2="-7.62" width="0.1524" layer="91"/>
 <junction x="-83.82" y="-7.62"/>
+</segment>
+<segment>
+<pinref part="LT3579_IC_" gate="G$1" pin="SYNC"/>
+<wire x1="17.78" y1="12.7" x2="25.4" y2="12.7" width="0.1524" layer="91"/>
+<label x="25.4" y="12.7" size="1.778" layer="95"/>
 </segment>
 </net>
@@
 <wire x1="22.86" y1="-43.18" x2="27.94" y2="-43.18" width="0.1524" layer="91"/>
 <junction x="22.86" y="-33.02"/>
+<junction x="22.86" y="0"/>
+<junction x="22.86" y="-2.54"/>
+<junction x="22.86" y="-5.08"/>
+<junction x="22.86" y="-7.62"/>
+<junction x="-22.86" y="-7.62"/>
+<junction x="-22.86" y="-5.08"/>
+<junction x="-22.86" y="-2.54"/>
+<junction x="-22.86" y="0"/>
 </segment>
 <segment>
@@
 <wire x1="-83.82" y1="-22.86" x2="-83.82" y2="-5.08" width="0.1524" layer="91"/>
 <junction x="-83.82" y="-5.08"/>
+</segment>
+<segment>
+<pinref part="LT3579_IC_1" gate="G$1" pin="SYNC"/>
+<wire x1="17.78" y1="15.24" x2="25.4" y2="15.24" width="0.1524" layer="91"/>
+<label x="25.4" y="15.24" size="1.778" layer="95"/>
 </segment>
 </net>
@@
 <wire x1="22.86" y1="-43.18" x2="27.94" y2="-43.18" width="0.1524" layer="91"/>
 <junction x="22.86" y="-33.02"/>
+<junction x="-22.86" y="0"/>
+<junction x="-22.86" y="-2.54"/>
+<junction x="-22.86" y="-5.08"/>
+<junction x="-22.86" y="-7.62"/>
+<junction x="22.86" y="-7.62"/>
+<junction x="22.86" y="-5.08"/>
+<junction x="22.86" y="-2.54"/>
+<junction x="22.86" y="0"/>
 </segment>
 <segment>
@@
 <junction x="-83.82" y="-5.08"/>
 </segment>
-</net>
+<segment>
+<pinref part="LT3579_IC_2" gate="G$1" pin="SYNC"/>
+<wire x1="17.78" y1="15.24" x2="25.4" y2="15.24" width="0.1524" layer="91"/>
+<label x="25.4" y="15.24" size="1.778" layer="95"/>
+</segment>
+</net>

Commit message: Added Board Layout. Initial Board Layout done.
Parts:
- renumbered R_RB_1 to R_FB_1
Connections:
- net 0: now also L1L2_.4, L1L2_1.4, L1L2_2.4, TP_GND1_.1, TP_GND1_1.1, TP_GND1_2.1, TP_GND2_.1, TP_GND2_1.1, TP_GND2_2.1, TP_GND3_.1, TP_GND3_1.1, TP_GND3_2.1, TP_GND4_.1, TP_GND4_1.1, TP_GND4_2.1
- net CH_GND: now also TP_CH_GND_.1, TP_CH_GND_1.1, TP_CH_GND_2.1
- net CLK_: now also TP_CLK_.1
- net CLK_1: now also TP_CLK_1.1
- net CLK_2: now also TP_CLK_2.1
- net FAULT_: now also TP_FAULT_.1
- net FAULT_1: now also TP_FAULT_1.1
- net FAULT_2: now also TP_FAULT_2.1
- net GATE_: now also TP_GATE_.1
- net GATE_1: now also TP_GATE_1.1
- net GATE_2: now also TP_GATE_2.1
- net GND: now also TP_GND_.1, TP_GND_1.1, TP_GND_2.1
- net N$1: now also L1L2_1.2, TP_D1_1.1
- net N$13: now also TP_FB_.1
- net N$3: now also TP_FB_1.1
- net N$5: now also L1L2_2.2, TP_D1_2.1
- net N$7: now also TP_FB_2.1
- net N$9: now also L1L2_.2, TP_D1_.1
- net RT_: now also TP_RT_.1
- net RT_1: now also TP_RT_1.1
- net RT_2: now also TP_RT_2.1
- net SHDN_: now also TP_SHDN_.1
- net SHDN_1: now also TP_SHDN_1.1
- net SHDN_2: now also TP_SHDN_2.1
- net SS_: now also TP_SS_.1
- net SS_1: now also TP_SS_1.1
- net SS_2: now also TP_SS_2.1
- net SW1-2_: now also L1L2_.1, TP_SW_.1
- net SW1-2_1: now also L1L2_1.1, TP_SW_1.1
- net SW1-2_2: now also L1L2_2.1, TP_SW_2.1
- net VC_: now also TP_CF_.1
- net VC_1: now also TP_CF_1.1
- net VC_2: now also TP_CF_2.1
- net VIN: now also L1L2_.3, L1L2_1.3, L1L2_2.3, TP_IN_.1, TP_IN_1.1, TP_IN_2.1
- net VOUT_: now also TP_OUT_.1
- net VOUT_1: now also TP_OUT_1.1
- net VOUT_2: now also TP_OUT_2.1
Other:
- moved on the sheet: C_C_, C_C_1, R_C_, R_FAULT_1, TP_CF_, TP_FAULT_1, TP_FB_2

Commit message: new files
Parts:
- added C_68N_FILTER_, C_68N_FILTER_1, C_68N_FILTER_2: CEU4J2X7R1H683K125AE, SamacSys_Parts:CEU4J2X7R1H683K125AE
- added C_LDO_IN_, C_LDO_IN_1, C_LDO_IN_2: CGA3E1X7R1V105K080AC, SamacSys_Parts:CGA3E1X7R1V105K080AC
- added C_LDO_OUT_, C_LDO_OUT_1, C_LDO_OUT_2: JMK107BB7475KA-T, SamacSys_Parts:JMK107BB7475KA-T
- added C_LS_, C_LS_1, C_LS_2: CGA2B2C0G1H102J050BE, SamacSys_Parts:CGA2B2C0G1H102J050BE
- added LDO_, LDO_1, LDO_2: LDL1117S33R, SamacSys_Parts:LDL1117S33R
- added LED_, LED_1, LED_2: APTD1608LCGCK, SamacSys_Parts:APTD1608LCGCK
- added NMOS_LDO_, NMOS_LDO_1, NMOS_LDO_2: RTR025N05HZGTL, SamacSys_Parts:RTR025N05HZGTL
- added R_10K_FILTER_, R_10K_FILTER_1, R_10K_FILTER_2: AC0805DR-0710KL, AC0805DR-0710KL:AC0805DR-0710KL
- added R_20K_LED1_: ERJ-2RKF2002X, SamacSys_Parts:ERJ-2RKF2002X
- added R_5.6K_LED2_: ERA-2ARB562X, SamacSys_Parts:ERA-2ARB562X
- added R_5K_FILTER_\, R_5K_FILTER_\1, R_5K_FILTER_\2: RT1206BRD075KL, SamacSys_Parts:RT1206BRD075KL
- added R_LED_10K_1, R_LED_10K_2, R_LS_DRAIN_, R_LS_DRAIN_1, R_LS_DRAIN_2: MCS0402MD1002DE000, SamacSys_Parts:MCS0402MD1002DE000
- added R_LS_GATE_, R_LS_GATE_1, R_LS_GATE_2: AT0805FRE07100KL, AT0805FRE07100KL:AT0805FRE07100KL
- added TP_CLK_FILTER_, TP_CLK_FILTER_1, TP_CLK_FILTER_2, TP_FAULT_LS_, TP_FAULT_LS_1, TP_FAULT_LS_2, TP_LDO_OUT_, TP_LDO_OUT_1, TP_LDO_OUT_2: S1751-46R, S1751-46R:S1751-46R
Connections:
- new net CLK_FILTER_OUT_: 12P_OUTPUT_CONNECTOR1.6, C_68N_FILTER_.1, R_10K_FILTER_.2, R_5K_FILTER_\.1, TP_CLK_FILTER_.1
- new net CLK_FILTER_OUT_1: 12P_OUTPUT_CONNECTOR1.4, C_68N_FILTER_1.1, R_10K_FILTER_1.2, R_5K_FILTER_\1.1, TP_CLK_FILTER_1.1
- new net CLK_FILTER_OUT_2: 12P_OUTPUT_CONNECTOR1.2, C_68N_FILTER_2.1, R_10K_FILTER_2.2, R_5K_FILTER_\2.1, TP_CLK_FILTER_2.1
- new net FAULT_LS_OUT_: 12P_OUTPUT_CONNECTOR1.5, C_LS_.1, NMOS_LDO_.DRAIN, R_LS_DRAIN_.1, TP_FAULT_LS_.1
- new net FAULT_LS_OUT_1: 12P_OUTPUT_CONNECTOR1.3, C_LS_1.1, NMOS_LDO_1.DRAIN, R_LS_DRAIN_1.1, TP_FAULT_LS_1.1
- new net FAULT_LS_OUT_2: 12P_OUTPUT_CONNECTOR1.1, C_LS_2.1, NMOS_LDO_2.DRAIN, R_LS_DRAIN_2.1, TP_FAULT_LS_2.1
- new net LDO_OUT_: C_LDO_OUT_.1, LDO_.VOUT_1, LDO_.VOUT_2, R_LS_DRAIN_.2, TP_LDO_OUT_.1
- new net LDO_OUT_1: C_LDO_OUT_1.1, LDO_1.VOUT_1, LDO_1.VOUT_2, R_LS_DRAIN_1.2, TP_LDO_OUT_1.1
- new net LDO_OUT_2: C_LDO_OUT_2.1, LDO_2.VOUT_1, LDO_2.VOUT_2, R_LS_DRAIN_2.2, TP_LDO_OUT_2.1
- new net N$10: NMOS_LDO_1.GATE, R_LS_GATE_1.2
- new net N$11: LED_1.A, R_LED_10K_1.2
- new net N$12: R_20K_LED1_.1, R_5.6K_LED2_.1
- new net N$14: NMOS_LDO_2.GATE, R_LS_GATE_2.2
- new net N$15: LED_.A, R_5.6K_LED2_.2
- new net N$16: LED_2.A, R_LED_10K_2.2
- new net N$8: NMOS_LDO_.GATE, R_LS_GATE_.2
- net 0: now also C_68N_FILTER_.2, C_68N_FILTER_1.2, C_68N_FILTER_2.2, C_LDO_IN_.2, C_LDO_IN_1.2, C_LDO_IN_2.2, C_LDO_OUT_.2, C_LDO_OUT_1.2, C_LDO_OUT_2.2, C_LS_.2, C_LS_1.2, C_LS_2.2, LED_.K, LED_1.K, LED_2.K, NMOS_LDO_.SOURCE, NMOS_LDO_1.SOURCE, NMOS_LDO_2.SOURCE, R_5K_FILTER_\.2, R_5K_FILTER_\1.2, R_5K_FILTER_\2.2
- net CLK_: now also R_10K_FILTER_.1; no longer 12P_OUTPUT_CONNECTOR1.6
- net CLK_1: now also R_10K_FILTER_1.1; no longer 12P_OUTPUT_CONNECTOR1.4
- net CLK_2: now also R_10K_FILTER_2.1; no longer 12P_OUTPUT_CONNECTOR1.2
- net FAULT_: now also R_LS_GATE_.1; no longer 12P_OUTPUT_CONNECTOR1.5
- net FAULT_1: now also R_LS_GATE_1.1; no longer 12P_OUTPUT_CONNECTOR1.3
- net FAULT_2: now also R_LS_GATE_2.1; no longer 12P_OUTPUT_CONNECTOR1.1
- net GND: now also LDO_.GND, LDO_1.GND, LDO_2.GND
- net VIN: now also C_LDO_IN_.1, C_LDO_IN_1.1, C_LDO_IN_2.1, LDO_.VIN, LDO_1.VIN, LDO_2.VIN
- net VOUT_: now also R_20K_LED1_.2
- net VOUT_1: now also R_LED_10K_1.1
- net VOUT_2: now also R_LED_10K_2.1
Other:
- note added: "13V -> 3.3V output"
- note added: "13V FAULT logic level -> 3.3V Logic Level"
- note added: "20K + 5.6K Series Resistance"
- note added: "Filter to convert pulse signal to DC"
- moved on the sheet: R_SHUNT_GND_, TP_CH_GND_, TP_GND_

Commit message: Removed and replaced files
Parts:
- removed C_LDO_IN_1, C_LDO_IN_2: CGA3E1X7R1V105K080AC, SamacSys_Parts:CGA3E1X7R1V105K080AC
- removed C_LDO_OUT_1, C_LDO_OUT_2: JMK107BB7475KA-T, SamacSys_Parts:JMK107BB7475KA-T
- removed LDO_1, LDO_2: LDL1117S33R, SamacSys_Parts:LDL1117S33R
- removed TP_LDO_OUT_1, TP_LDO_OUT_2: S1751-46R, S1751-46R:S1751-46R
- added PMOS_REVERSE_V_PROTECTION: DMP3015LSSQ-13, DMP3015LSSQ-13:DMP3015LSSQ-13
- D1_, D1_1, D1_2: value MBRS360T3G -> MBRS330T3G; device SamacSys_Parts:MBRS360T3G -> SamacSys_Parts:MBRS330T3G
- NMOS_LDO_, NMOS_LDO_1, NMOS_LDO_2: value RTR025N05HZGTL -> RSR025N03HZGTL; device SamacSys_Parts:RTR025N05HZGTL -> SamacSys_Parts:RSR025N03HZGTL
- R_GATE_, R_GATE_1, R_GATE_2: value AC0805DR-0710KL -> AC0805FR-0710KL; device AC0805DR-0710KL:AC0805DR-0710KL -> SamacSys_Parts:AC0805FR-0710KL
Connections:
- removed net LDO_OUT_1: C_LDO_OUT_1.1, LDO_1.VOUT_1, LDO_1.VOUT_2, R_LS_DRAIN_1.2, TP_LDO_OUT_1.1
- removed net LDO_OUT_2: C_LDO_OUT_2.1, LDO_2.VOUT_1, LDO_2.VOUT_2, R_LS_DRAIN_2.2, TP_LDO_OUT_2.1
- new net VIN_CONNECTOR: 4P_INPUT_CONNECTOR1.1, 4P_INPUT_CONNECTOR1.3, PMOS_REVERSE_V_PROTECTION.D1
- net 0: now also NMOS_LDO_.S, NMOS_LDO_1.S, NMOS_LDO_2.S, PMOS_REVERSE_V_PROTECTION.G1; no longer C_LDO_IN_1.2, C_LDO_IN_2.2, C_LDO_OUT_1.2, C_LDO_OUT_2.2, NMOS_LDO_.SOURCE, NMOS_LDO_1.SOURCE, NMOS_LDO_2.SOURCE
- net FAULT_LS_OUT_: now also NMOS_LDO_.D; no longer NMOS_LDO_.DRAIN
- net FAULT_LS_OUT_1: now also NMOS_LDO_1.D; no longer NMOS_LDO_1.DRAIN
- net FAULT_LS_OUT_2: now also NMOS_LDO_2.D; no longer NMOS_LDO_2.DRAIN
- net GND: no longer LDO_1.GND, LDO_2.GND
- net LDO_OUT_: now also R_LS_DRAIN_1.2, R_LS_DRAIN_2.2
- net N$10: now also NMOS_LDO_1.G; no longer NMOS_LDO_1.GATE
- net N$14: now also NMOS_LDO_2.G; no longer NMOS_LDO_2.GATE
- net N$8: now also NMOS_LDO_.G; no longer NMOS_LDO_.GATE
- net VIN: now also PMOS_REVERSE_V_PROTECTION.S1; no longer 4P_INPUT_CONNECTOR1.1, 4P_INPUT_CONNECTOR1.3, C_LDO_IN_1.1, C_LDO_IN_2.1, LDO_1.VIN, LDO_2.VIN
Other:
- moved on the sheet: C_68N_FILTER_, C_68N_FILTER_1, C_68N_FILTER_2, C_LDO_IN_, C_LDO_OUT_, C_LS_, C_LS_1, C_LS_2, LDO_, LED_, LED_1, NMOS_LDO_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

Commit message: Added and Replaced new files
Parts:
- removed C_DECOUPLE_CH_GND_1: CGA4F4C0G2W222J085AE, SamacSys_Parts:CGA4F4C0G2W222J085AE
- removed C_DECOUPLE_CH_GND_2: CGADN3X7R1E476M230LE, SamacSys_Parts:CGADN3X7R1E476M230LE
- added C_DEC_CH_GND_1: CGA4F4C0G2W222J085AE, SamacSys_Parts:CGA4F4C0G2W222J085AE
- added C_DEC_CH_GND_2: CGADN3X7R1E476M230LE, SamacSys_Parts:CGADN3X7R1E476M230LE
- added U$1, U$2, U$3, U$4: THROUGH_HOLE_, THROUGH_HOLE:THROUGH_HOLE_
Connections:
- removed net 0: C_68N_FILTER_.2, C_68N_FILTER_1.2, C_68N_FILTER_2.2, C_C_.2, C_C_1.2, C_C_2.2, C_F_.2, C_F_1.2, C_F_2.2, C_IN_1_.2, C_IN_1_1.2, C_IN_1_2.2, C_IN_2_.2, C_IN_2_1.2, C_IN_2_2.2, C_LDO_IN_.2, C_LDO_OUT_.2, C_LS_.2, C_LS_1.2, C_LS_2.2, C_OUT_1_.2, C_OUT_1_1.2, C_OUT_1_2.2, C_OUT_2_.2, C_OUT_2_1.2, C_OUT_2_2.2, C_OUT_3_.2, C_OUT_3_1.2, C_OUT_3_2.2, C_SS_.2, C_SS_1.2, C_SS_2.2, L1L2_.4, L1L2_1.4, L1L2_2.4, LED_.K, LED_1.K, LED_2.K, LT3579_IC_.EPAD, LT3579_IC_1.EPAD, LT3579_IC_2.EPAD, NMOS_LDO_.S, NMOS_LDO_1.S, NMOS_LDO_2.S, PMOS_REVERSE_V_PROTECTION.G1, R_5K_FILTER_\.2, R_5K_FILTER_\1.2, R_5K_FILTER_\2.2, R_T_.2, R_T_1.2, R_T_2.2, R_UVLO2_.1, R_UVLO2_1.1, R_UVLO2_2.1, TP_GND1_.1, TP_GND1_1.1, TP_GND1_2.1, TP_GND2_.1, TP_GND2_1.1, TP_GND2_2.1, TP_GND3_.1, TP_GND3_1.1, TP_GND3_2.1, TP_GND4_.1, TP_GND4_1.1, TP_GND4_2.1
- removed net GND: 12P_OUTPUT_CONNECTOR1.10, 12P_OUTPUT_CONNECTOR1.12, 12P_OUTPUT_CONNECTOR1.8, LDO_.GND, LT3579_IC_.SYNC, LT3579_IC_1.SYNC, LT3579_IC_2.SYNC, R_SHUNT_GND_.2, R_SHUNT_GND_1.2, R_SHUNT_GND_2.2, TP_GND_.1, TP_GND_1.1, TP_GND_2.1
- new net GND_: 12P_OUTPUT_CONNECTOR1.12, C_68N_FILTER_.2, C_C_.2, C_F_.2, C_IN_1_.2, C_IN_2_.2, C_LS_.2, C_OUT_1_.2, C_OUT_2_.2, C_OUT_3_.2, C_SS_.2, L1L2_.4, LED_.K, LT3579_IC_.EPAD, LT3579_IC_.SYNC, NMOS_LDO_.S, R_5K_FILTER_\.2, R_SHUNT_GND_.2, R_T_.2, R_UVLO2_.1, TP_GND1_.1, TP_GND2_.1, TP_GND3_.1, TP_GND4_.1, TP_GND_.1
- new net GND_1: 12P_OUTPUT_CONNECTOR1.10, C_68N_FILTER_1.2, C_C_1.2, C_F_1.2, C_IN_1_1.2, C_IN_2_1.2, C_LS_1.2, C_OUT_1_1.2, C_OUT_2_1.2, C_OUT_3_1.2, C_SS_1.2, L1L2_1.4, LED_1.K, LT3579_IC_1.EPAD, LT3579_IC_1.SYNC, NMOS_LDO_1.S, R_5K_FILTER_\1.2, R_SHUNT_GND_1.2, R_T_1.2, R_UVLO2_1.1, TP_GND1_1.1, TP_GND2_1.1, TP_GND3_1.1, TP_GND4_1.1, TP_GND_1.1
- new net GND_2: 12P_OUTPUT_CONNECTOR1.8, C_68N_FILTER_2.2, C_C_2.2, C_F_2.2, C_IN_1_2.2, C_IN_2_2.2, C_LS_2.2, C_OUT_1_2.2, C_OUT_2_2.2, C_OUT_3_2.2, C_SS_2.2, L1L2_2.4, LED_2.K, LT3579_IC_2.EPAD, LT3579_IC_2.SYNC, NMOS_LDO_2.S, R_5K_FILTER_\2.2, R_SHUNT_GND_2.2, R_T_2.2, R_UVLO2_2.1, TP_GND1_2.1, TP_GND2_2.1, TP_GND3_2.1, TP_GND4_2.1, TP_GND_2.1
- net CH_GND: now also C_DEC_CH_GND_1.1, C_DEC_CH_GND_2.1, C_LDO_IN_.2, C_LDO_OUT_.2, LDO_.GND, PMOS_REVERSE_V_PROTECTION.G1; no longer C_DECOUPLE_CH_GND_1.1, C_DECOUPLE_CH_GND_2.1
- net VIN: now also C_DEC_CH_GND_1.2, C_DEC_CH_GND_2.2; no longer C_DECOUPLE_CH_GND_1.2, C_DECOUPLE_CH_GND_2.2
Other:
- note added: "12-Pin connector carrying Power and Signal out of the board. Will mate with a male connector on the board enclosure."
- note added: "Chasis GND is the car frame."
- note added: "Feedback Resistor (R_B) sets the output voltage of the circuit."
- note added: "Filter to convert pulse signal to DC for MCU. Cutoff set at 700Hz. Gain = 1/3."
- note added: "GND test points to be placed near signal and pwr test points."
- note added: "Holes for mounting board to enclosures. For bolt size of 1/16""
- note added: "Input"
- note added: "Input Capacitors to reduce ripple voltage from battery."
- note added: "LDO to step down battery voltage to 3.3V for the lofig level shifter"
- note added: "Logic Level Shifter. 13V to 3.3V for MCU."
- note added: "Oscillator Timing Resistor (R_T) sets the operating freqeuncy of LT3579. Operating Frequency is set to 700KHz."
- note added: "Output Capacitors to reduce voltage ripple"
- note added: "PMOS for output disconnect. GATE pin turns off or on the PMOS."
- note added: "PMOS for reverse voltage protection. If battery is plugged in the wrong way."
- note added: "PWR on light indicator."
- note added: "Pull up resistor for the FAULT indicator pin. FAULT can be pulled low externally or internally."
- note added: "R_C,C_C, and C_F form a recictor-capacitor network to compensate the voltage feedback loop in the LT3579."
- note added: "Shunt resistor to measure the difference between chasis GND and signal GND."
- note added: "Soft-start: C_SS is in series w/ integrated 250K resistor of LT3579. Determins the charging and discharing rate when the part shutsdown."
- note added: "Voltage divider by R_UVLO1/2 set the low voltage lockout for the LT3579. UVLO is set at 10V. LT3579 will turn off, if this min threshold is not met to protect battery."
- note removed: "13V FAULT logic level -> 3.3V Logic Level"
- note removed: "Connector for all voltage outputs, GNDs, CLK, and Faults."
- note removed: "Filter to convert pulse signal to DC"
- note removed: "Shunt resistor to measure difference between GNDS."
- note removed: "This will mate with the male connector on the enclosure."
- moved on the sheet: 12P_OUTPUT_CONNECTOR1, 4P_INPUT_CONNECTOR1, C_1_, C_68N_FILTER_, C_68N_FILTER_1, C_68N_FILTER_2, C_C_, C_C_1, C_C_2, C_F_, C_F_1, C_F_2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
