File: LT3579-SEPIC-EAGLE-Project/LT3579_SEPIC_Test_Bench.sch (EAGLE design)
At the start: 160 parts

Commit message: Added new FIles
Parts:
- removed C_68N_FILTER_, C_68N_FILTER_1, C_68N_FILTER_2: CEU4J2X7R1H683K125AE, SamacSys_Parts:CEU4J2X7R1H683K125AE
- removed C_DECOUPLE_CH_GND_1: CGA4F4C0G2W222J085AE, SamacSys_Parts:CGA4F4C0G2W222J085AE
- removed C_DECOUPLE_CH_GND_2: CGADN3X7R1E476M230LE, SamacSys_Parts:CGADN3X7R1E476M230LE
- removed R_10K_FILTER_, R_10K_FILTER_1, R_10K_FILTER_2: AC0805DR-0710KL, AC0805DR-0710KL:AC0805DR-0710KL
- removed R_5K_FILTER_\, R_5K_FILTER_\1, R_5K_FILTER_\2: RT1206BRD075KL, SamacSys_Parts:RT1206BRD075KL
- removed TP_CLK_FILTER_, TP_CLK_FILTER_1, TP_CLK_FILTER_2: S1751-46R, S1751-46R:S1751-46R
- added C_68N_F_, C_68N_F_1, C_68N_F_2: CEU4J2X7R1H683K125AE, SamacSys_Parts:CEU4J2X7R1H683K125AE
- added C_DEC_CH_GND_1: CGA4F4C0G2W222J085AE, SamacSys_Parts:CGA4F4C0G2W222J085AE
- added C_DEC_CH_GND_2: CGADN3X7R1E476M230LE, SamacSys_Parts:CGADN3X7R1E476M230LE
- added R_10K_F_, R_10K_F_1, R_10K_F_2: AC0805DR-0710KL, AC0805DR-0710KL:AC0805DR-0710KL
- added R_5K_F_, R_5K_F_1, R_5K_F_2: RT1206BRD075KL, SamacSys_Parts:RT1206BRD075KL
- added TP_CLK_F_, TP_CLK_F_1, TP_CLK_F_2: S1751-46R, S1751-46R:S1751-46R
- added U$1, U$2, U$3, U$4: THROUGH_HOLE_, THROUGH_HOLE:THROUGH_HOLE_
Connections:
- removed net 0: C_68N_FILTER_.2, C_68N_FILTER_1.2, C_68N_FILTER_2.2, C_C_.2, C_C_1.2, C_C_2.2, C_F_.2, C_F_1.2, C_F_2.2, C_IN_1_.2, C_IN_1_1.2, C_IN_1_2.2, C_IN_2_.2, C_IN_2_1.2, C_IN_2_2.2, C_LDO_IN_.2, C_LDO_OUT_.2, C_LS_.2, C_LS_1.2, C_LS_2.2, C_OUT_1_.2, C_OUT_1_1.2, C_OUT_1_2.2, C_OUT_2_.2, C_OUT_2_1.2, C_OUT_2_2.2, C_OUT_3_.2, C_OUT_3_1.2, C_OUT_3_2.2, C_SS_.2, C_SS_1.2, C_SS_2.2, L1L2_.4, L1L2_1.4, L1L2_2.4, LED_.K, LED_1.K, LED_2.K, LT3579_IC_.EPAD, LT3579_IC_1.EPAD, LT3579_IC_2.EPAD, NMOS_LDO_.S, NMOS_LDO_1.S, NMOS_LDO_2.S, PMOS_REVERSE_V_PROTECTION.G1, R_5K_FILTER_\.2, R_5K_FILTER_\1.2, R_5K_FILTER_\2.2, R_T_.2, R_T_1.2, R_T_2.2, R_UVLO2_.1, R_UVLO2_1.1, R_UVLO2_2.1, TP_GND1_.1, TP_GND1_1.1, TP_GND1_2.1, TP_GND2_.1, TP_GND2_1.1, TP_GND2_2.1, TP_GND3_.1, TP_GND3_1.1, TP_GND3_2.1, TP_GND4_.1, TP_GND4_1.1, TP_GND4_2.1
- removed net GND: 12P_OUTPUT_CONNECTOR1.10, 12P_OUTPUT_CONNECTOR1.12, 12P_OUTPUT_CONNECTOR1.8, LDO_.GND, LT3579_IC_.SYNC, LT3579_IC_1.SYNC, LT3579_IC_2.SYNC, R_SHUNT_GND_.2, R_SHUNT_GND_1.2, R_SHUNT_GND_2.2, TP_GND_.1, TP_GND_1.1, TP_GND_2.1
- new net GND_: 12P_OUTPUT_CONNECTOR1.12, C_68N_F_.2, C_C_.2, C_F_.2, C_IN_1_.2, C_IN_2_.2, C_LS_.2, C_OUT_1_.2, C_OUT_2_.2, C_OUT_3_.2, C_SS_.2, L1L2_.4, LED_.K, LT3579_IC_.EPAD, LT3579_IC_.SYNC, NMOS_LDO_.S, R_5K_F_.2, R_SHUNT_GND_.2, R_T_.2, R_UVLO2_.1, TP_GND1_.1, TP_GND2_.1, TP_GND3_.1, TP_GND4_.1, TP_GND_.1
- new net GND_1: 12P_OUTPUT_CONNECTOR1.10, C_68N_F_1.2, C_C_1.2, C_F_1.2, C_IN_1_1.2, C_IN_2_1.2, C_LS_1.2, C_OUT_1_1.2, C_OUT_2_1.2, C_OUT_3_1.2, C_SS_1.2, L1L2_1.4, LED_1.K, LT3579_IC_1.EPAD, LT3579_IC_1.SYNC, NMOS_LDO_1.S, R_5K_F_1.2, R_SHUNT_GND_1.2, R_T_1.2, R_UVLO2_1.1, TP_GND1_1.1, TP_GND2_1.1, TP_GND3_1.1, TP_GND4_1.1, TP_GND_1.1
- new net GND_2: 12P_OUTPUT_CONNECTOR1.8, C_68N_F_2.2, C_C_2.2, C_F_2.2, C_IN_1_2.2, C_IN_2_2.2, C_LS_2.2, C_OUT_1_2.2, C_OUT_2_2.2, C_OUT_3_2.2, C_SS_2.2, L1L2_2.4, LED_2.K, LT3579_IC_2.EPAD, LT3579_IC_2.SYNC, NMOS_LDO_2.S, R_5K_F_2.2, R_SHUNT_GND_2.2, R_T_2.2, R_UVLO2_2.1, TP_GND1_2.1, TP_GND2_2.1, TP_GND3_2.1, TP_GND4_2.1, TP_GND_2.1
- net CH_GND: now also C_DEC_CH_GND_1.1, C_DEC_CH_GND_2.1, C_LDO_IN_.2, C_LDO_OUT_.2, LDO_.GND, PMOS_REVERSE_V_PROTECTION.G1; no longer C_DECOUPLE_CH_GND_1.1, C_DECOUPLE_CH_GND_2.1
- net CLK_: now also R_10K_F_.1; no longer R_10K_FILTER_.1
- net CLK_1: now also R_10K_F_1.1; no longer R_10K_FILTER_1.1
- net CLK_2: now also R_10K_F_2.1; no longer R_10K_FILTER_2.1
- net CLK_FILTER_OUT_: now also C_68N_F_.1, R_10K_F_.2, R_5K_F_.1, TP_CLK_F_.1; no longer C_68N_FILTER_.1, R_10K_FILTER_.2, R_5K_FILTER_\.1, TP_CLK_FILTER_.1
- net CLK_FILTER_OUT_1: now also C_68N_F_1.1, R_10K_F_1.2, R_5K_F_1.1, TP_CLK_F_1.1; no longer C_68N_FILTER_1.1, R_10K_FILTER_1.2, R_5K_FILTER_\1.1, TP_CLK_FILTER_1.1
- net CLK_FILTER_OUT_2: now also C_68N_F_2.1, R_10K_F_2.2, R_5K_F_2.1, TP_CLK_F_2.1; no longer C_68N_FILTER_2.1, R_10K_FILTER_2.2, R_5K_FILTER_\2.1, TP_CLK_FILTER_2.1
- net VIN: now also C_DEC_CH_GND_1.2, C_DEC_CH_GND_2.2; no longer C_DECOUPLE_CH_GND_1.2, C_DECOUPLE_CH_GND_2.2
Other:
- note added: "12-Pin connector carrying Power and Signal out of the board. Will mate with a male connector on the board enclosure."
- note added: "Chasis GND is the car frame."
- note added: "Feedback Resistor (R_B) sets the output voltage of the circuit."
- note added: "Filter to convert pulse signal to DC for MCU. Cutoff set at 700Hz. Gain = 1/3."
- note added: "GND test points to be placed near signal and pwr test points."
- note added: "Holes for mounting board to enclosures. For bolt size of 1/16""
- note added: "Input"
- note added: "Input Capacitors to reduce ripple voltage from battery."
- note added: "LDO to step down battery voltage to 3.3V for the lofig level shifter"
- note added: "Logic Level Shifter. 13V to 3.3V for MCU."
- note added: "Oscillator Timing Resistor (R_T) sets the operating freqeuncy of LT3579. Operating Frequency is set to 700KHz."
- note added: "Output Capacitors to reduce voltage ripple"
- note added: "PMOS for output disconnect. GATE pin turns off or on the PMOS."
- note added: "PMOS for reverse voltage protection. If battery is plugged in the wrong way."
- note added: "PWR on light indicator."
- note added: "Pull up resistor for the FAULT indicator pin. FAULT can be pulled low externally or internally."
- note added: "R_C,C_C, and C_F form a recictor-capacitor network to compensate the voltage feedback loop in the LT3579."
- note added: "Shunt resistor to measure the difference between chasis GND and signal GND."
- note added: "Soft-start: C_SS is in series w/ integrated 250K resistor of LT3579. Determins the charging and discharing rate when the part shutsdown."
- note added: "Voltage divider by R_UVLO1/2 set the low voltage lockout for the LT3579. UVLO is set at 10V. LT3579 will turn off, if this min threshold is not met to protect battery."
- note removed: "13V FAULT logic level -> 3.3V Logic Level"
- note removed: "Connector for all voltage outputs, GNDs, CLK, and Faults."
- note removed: "Filter to convert pulse signal to DC"
- note removed: "Shunt resistor to measure difference between GNDS."
- note removed: "This will mate with the male connector on the enclosure."
- moved on the sheet: 12P_OUTPUT_CONNECTOR1, 4P_INPUT_CONNECTOR1, C_1_, C_C_, C_C_1, C_C_2, C_F_, C_F_1, C_F_2, C_IN_1_, C_IN_2_, C_LDO_IN_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
